File: PCB/Control PCb.brd (EAGLE design)
At the start: 45.7 x 76.2 mm, 7 parts

Commit message: PCB files etc
Parts:
- added D1: LED_GREEN, RJC-2:CHIP_LED0805
- added J6: (no value), SparkFun-Connectors:1X01_OFFSET
- added J7: (no value), SparkFun-Connectors:1X02_LOCK_LONGPADS
- added Q1: DMP2305U-7, RJC-2:SOT23
- added Q2, Q3: BSS123, RJC-2:SOT23
- added R2, R3, R4, R5: 0, RJC-2:0805
- moved R1 7.01 mm to (32.6, 22.0)
- moved J4 3.98 mm to (42.6, 19.2), turned to 270 degrees
Connections:
- new net N$10: J2.4, R5.1
- new net N$11: J6.1, Q3.3
- new net N$5: Q1.1, Q2.3, R2.1
- new net N$6: J4.1, Q1.2, R3.1
- new net N$7: D1.A, R3.2
- new net N$8: Q3.1, R4.2, R5.2
- new net N$9: J2.5, R4.1
- net +5V: now also J7.2, Q1.3, R2.2
- net GND: now also D1.C, J7.1, Q2.2, Q3.2
- net N$2: now also Q2.1; no longer J4.1
Routing:
- net +5V: track 22.4 -> 42.0 mm
- net N$10: track 0.00 -> 12.1 mm
- net N$6: track 0.00 -> 10.1 mm
- net N$5: track 0.00 -> 9.91 mm
- net N$9: track 0.00 -> 8.89 mm
- net N$1: track 11.2 -> 3.96 mm
- net N$8: track 0.00 -> 3.92 mm
- net N$11: track 0.00 -> 2.94 mm
- net N$7: track 0.00 -> 2.05 mm

Commit message: SW
Parts:
- moved J5 11.7 mm to (5.08, 65.0), turned to 270 degrees
Routing:
- net N$4: track 62.0 -> 45.2 mm
- net N$3: track 52.2 -> 66.2 mm
- net +3V3: track 41.4 -> 42.4 mm
Changed lines of the file:
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@@
 <setting verticaltext="up"/>
 </settings>
-<grid distance="10" unitdist="mil" unit="mil" style="lines" multiple="1" display="yes" altdistance="5" altunitdist="mil" altunit="mil"/>
+<grid distance="100" unitdist="mil" unit="mm" style="lines" multiple="1" display="yes" altdistance="5" altunitdist="mil" altunit="mil"/>
 <layers>
 <layer number="1" name="Top" color="4" fill="1" visible="yes" active="yes"/>
@@
 <layer number="45" name="Holes" color="7" fill="1" visible="yes" active="yes"/>
 <layer number="46" name="Milling" color="3" fill="1" visible="no" active="yes"/>
-<layer number="47" name="Measures" color="7" fill="1" visible="no" active="yes"/>
+<layer number="47" name="Measures" color="7" fill="1" visible="yes" active="yes"/>
 <layer number="48" name="Document" color="7" fill="1" visible="yes" active="yes"/>
 <layer number="49" name="Reference" color="7" fill="1" visible="yes" active="yes"/>
@@
 <wire x1="0" y1="76.2" x2="0" y2="0" width="0" layer="20"/>
 <hole x="40.64" y="71.12" drill="3.2"/>
-<hole x="12.7" y="71.12" drill="3.2"/>
+<hole x="5.08" y="71.12" drill="3.2"/>
 <hole x="5.08" y="5.08" drill="3.2"/>
 <hole x="40.64" y="5.08" drill="3.2"/>
+<hole x="26.67" y="66.294" drill="2.794"/>
+<hole x="26.67" y="45.974" drill="2.794"/>
 </plain>
 <attributes>
@@
 <attribute name="VALUE" x="43.86" y="20.43" size="0.6096" layer="27" font="vector" ratio="20" rot="R270"/>
 </element>
-<element name="J5" library="SparkFun-Connectors" library_urn="urn:adsk.eagle:library:513" package="1X08_LOCK_LONGPADS" package3d_urn="urn:adsk.eagle:package:38140/1" value="" x="5.08" y="53.34" smashed="yes" rot="R90">
-<attribute name="NAME" x="3.302" y="52.451" size="0.6096" layer="25" font="vector" ratio="20" rot="R90"/>
-<attribute name="VALUE" x="7.366" y="52.197" size="0.6096" layer="27" font="vector" ratio="20" rot="R90"/>
+<element name="J5" library="SparkFun-Connectors" library_urn="urn:adsk.eagle:library:513" package="1X08_LOCK_LONGPADS" package3d_urn="urn:adsk.eagle:package:38140/1" value="" x="5.08" y="65.024" smashed="yes" rot="R270">
+<attribute name="NAME" x="6.858" y="65.913" size="0.6096" layer="25" font="vector" ratio="20" rot="R270"/>
+<attribute name="VALUE" x="2.794" y="66.167" size="0.6096" layer="27" font="vector" ratio="20" rot="R270"/>
 </element>
 <element name="R1" library="RJC-2" library_urn="urn:adsk.eagle:library:33162582" package="0805" package3d_urn="urn:adsk.eagle:package:33163805/3" value="0" x="32.59" y="22.04" smashed="yes" rot="MR180">
@@
 <contactref element="Q3" pad="2"/>
 <contactref element="J7" pad="1"/>
+<wire x1="5.334" y1="27.94" x2="28.067" y2="27.94" width="0" layer="19" extent="1-1"/>
 </signal>
 <signal name="+3V3">
 <contactref element="J1" pad="3"/>
 <contactref element="J5" pad="2"/>
-<wire x1="5.207" y1="55.88" x2="10.12" y2="55.88" width="1.27" layer="16"/>
-<wire x1="10.12" y1="55.88" x2="11.9" y2="54.1" width="1.27" layer="16"/>
-<wire x1="11.9" y1="54.1" x2="11.9" y2="28.1" width="1.27" layer="16"/>
-<wire x1="11.9" y1="28.1" x2="9.2" y2="25.4" width="1.27" layer="16"/>
-<wire x1="9.2" y1="25.4" x2="5.08" y2="25.4" width="1.27" layer="16"/>
+<wire x1="4.953" y1="62.484" x2="3.048" y2="62.484" width="1.016" layer="16"/>
+<wire x1="3.048" y1="62.484" x2="1.778" y2="61.214" width="1.016" layer="16"/>
+<wire x1="1.778" y1="61.214" x2="1.778" y2="26.162" width="1.016" layer="16"/>
+<wire x1="1.778" y1="26.162" x2="2.54" y2="25.4" width="1.016" layer="16"/>
+<wire x1="2.54" y1="25.4" x2="5.08" y2="25.4" width="1.016" layer="16"/>
 </signal>
 <signal name="+5V">
@@
 <contactref element="J5" pad="3"/>
 <contactref element="J1" pad="2"/>
-<wire x1="4.953" y1="58.42" x2="12.98" y2="58.42" width="1.27" layer="16"/>
-<wire x1="12.98" y1="58.42" x2="14.7" y2="56.7" width="1.27" layer="16"/>
-<wire x1="14.7" y1="56.7" x2="14.7" y2="25.5" width="1.27" layer="16"/>
-<wire x1="14.7" y1="25.5" x2="12" y2="22.8" width="1.27" layer="16"/>
-<wire x1="12" y1="22.8" x2="5.394" y2="22.8" width="1.27" layer="16"/>
 <wire x1="5.394" y1="22.8" x2="5.334" y2="22.86" width="1.27" layer="16"/>
+<wire x1="10.922" y1="59.944" x2="12.192" y2="58.674" width="1.016" layer="16"/>
+<wire x1="10.922" y1="59.944" x2="5.207" y2="59.944" width="1.016" layer="16"/>
+<wire x1="12.192" y1="19.05" x2="10.922" y2="17.78" width="1.016" layer="16"/>
+<wire x1="10.922" y1="17.78" x2="2.286" y2="17.78" width="1.016" layer="16"/>
+<wire x1="2.286" y1="17.78" x2="1.778" y2="18.288" width="1.016" layer="16"/>
+<wire x1="1.778" y1="18.288" x2="1.778" y2="22.352" width="1.016" layer="16"/>
+<wire x1="2.226" y1="22.8" x2="5.394" y2="22.8" width="1.016" layer="16"/>
+<wire x1="12.192" y1="58.674" x2="12.192" y2="19.05" width="1.016" layer="16"/>
+<wire x1="1.778" y1="22.352" x2="2.226" y2="22.8" width="1.016" layer="16"/>
 </signal>
 <signal name="N$4">
 <contactref element="J5" pad="4"/>
 <contactref element="J1" pad="1"/>
-<wire x1="5.207" y1="60.96" x2="15.14" y2="60.96" width="1.27" layer="16"/>
-<wire x1="15.14" y1="60.96" x2="17.5" y2="58.6" width="1.27" layer="16"/>
-<wire x1="17.5" y1="58.6" x2="17.5" y2="23.7" width="1.27" layer="16"/>
-<wire x1="17.5" y1="23.7" x2="14.1" y2="20.3" width="1.27" layer="16"/>
-<wire x1="14.1" y1="20.3" x2="5.1" y2="20.3" width="1.27" layer="16"/>
 <wire x1="5.1" y1="20.3" x2="5.08" y2="20.32" width="1.27" layer="16"/>
+<wire x1="4.953" y1="57.404" x2="8.382" y2="57.404" width="1.016" layer="16"/>
+<wire x1="8.87" y1="20.3" x2="5.1" y2="20.3" width="1.016" layer="16"/>
+<wire x1="8.382" y1="57.404" x2="9.652" y2="56.134" width="1.016" layer="16"/>
+<wire x1="9.652" y1="56.134" x2="9.652" y2="21.082" width="1.016" layer="16"/>
+<wire x1="9.652" y1="21.082" x2="8.87" y2="20.3" width="1.016" layer="16"/>
 </signal>
 <signal name="N$2">
